File: Evelope Follower/v1/envelope_follower_1.brd (EAGLE design)
At the start: 160 x 100 mm, 18 parts, among them J1 MJ-3536N, J2 MJ-3536N, J3 OSTVN03A150

Commit message: more changes
Parts:
- added TP1, TP2, TP3, TP4, TP5, TP6, TP7, TP8: (no value), roomready:TP_THM_1.6_S
- moved J2 79.4 mm to (46.1, 9.53)
- moved C2 41.7 mm to (21.6, 8.89)
- moved C3 41.7 mm to (24.1, 3.81)
- moved C4 41.7 mm to (39.1, 9.40)
- moved D1 41.7 mm to (22.6, 5.84)
- moved OP1 41.7 mm to (27.9, 8.89)
- moved R1 41.7 mm to (21.6, 11.4)
- moved R4 41.7 mm to (31.8, 5.08)
- moved R5 41.7 mm to (37.7, 6.22)
- moved R7 41.7 mm to (39.4, 12.1)
- moved C1 41.7 mm to (34.3, 8.89)
- moved D2 41.7 mm to (26.7, 3.81)
- moved R2 41.7 mm to (29.1, 3.81)
- moved R3 41.7 mm to (35.1, 5.97)
- moved R6 41.7 mm to (37.0, 9.40)
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Connections:
- net ENV: now also TP3.P$1
- net GND: now also TP2.P$1, TP4.P$1, TP8.P$1
- net LP_FILT: now also TP7.P$1
- net RECT: now also TP6.P$1
- net SRC: now also TP1.P$1
- net SRC_BUFF: now also TP5.P$1
Routing:
- net ENV: track 3.05 -> 27.4 mm
- net SRC: track 6.28 -> 19.6 mm
- net RECT: track 7.84 -> 20.5 mm, vias 0 -> 2
- net LP_FILT: track 8.61 -> 17.8 mm, vias 0 -> 2
- net +12V: track 2.63 -> 11.7 mm, vias 0 -> 2
- net SRC_BUFF: track 9.46 -> 18.5 mm
- net -12V: track 2.63 -> 11.6 mm
- added copper zone on layer 16, net GND
Other:
- board size 160 x 100 mm -> 59.7 x 20 mm

Commit message: ch-ch-ch-c
Parts:
- added J4: OSTVN02A150, roomready:OSTVN02A150
- R6: value 3.3k -> DNP
- moved R6 5.12 mm to (41.4, 6.86), turned to 180 degrees
- moved R5 3.27 mm to (37.0, 9.40), turned to 90 degrees
Connections:
- net LP_FILT: now also R5.2; no longer R6.1
- net N$2: now also J4.P$2
- net RECT: now also J4.P$1, R6.1; no longer R5.2
Routing:
- net RECT: track 20.5 -> 28.8 mm
- net N$2: track 1.79 -> 9.00 mm, vias 0 -> 1
Changed lines of the file:
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@@
 <attribute name="NAME" x="32.766" y="4.064" size="1.27" layer="25" rot="R180"/>
 </element>
-<element name="R5" library="roomready" library_urn="urn:adsk.eagle:library:9911636" package="R0603" package3d_urn="urn:adsk.eagle:package:7587835/3" value="3.3k" x="37.719" y="6.223" smashed="yes" rot="R270">
-<attribute name="NAME" x="38.354" y="6.858" size="1.27" layer="25" rot="R270"/>
-</element>
-<element name="R6" library="roomready" library_urn="urn:adsk.eagle:library:9911636" package="R0603" package3d_urn="urn:adsk.eagle:package:7587835/3" value="3.3k" x="36.957" y="9.398" smashed="yes" rot="R270">
-<attribute name="NAME" x="37.592" y="10.795" size="1.27" layer="25" rot="R90"/>
+<element name="R5" library="roomready" library_urn="urn:adsk.eagle:library:9911636" package="R0603" package3d_urn="urn:adsk.eagle:package:7587835/3" value="3.3k" x="36.957" y="9.398" smashed="yes" rot="R90">
+<attribute name="NAME" x="37.592" y="10.922" size="1.27" layer="25" rot="R90"/>
 </element>
 <element name="R7" library="roomready" library_urn="urn:adsk.eagle:library:9911636" package="R0603" package3d_urn="urn:adsk.eagle:package:7587835/3" value="2.2k" x="39.37" y="12.065" smashed="yes" rot="R180">
@@
 <element name="TP8" library="roomready" library_urn="urn:adsk.eagle:library:9911636" package="TP_THM_1.6_S" package3d_urn="urn:adsk.eagle:package:10068194/3" value="" x="34.29" y="2.54" smashed="yes">
 <attribute name="NAME" x="36.1188" y="2.032" size="1.27" layer="25"/>
+</element>
+<element name="J4" library="roomready" library_urn="urn:adsk.eagle:library:9911636" package="OSTVN02A150" package3d_urn="urn:adsk.eagle:package:12594929/2" value="OSTVN02A150" x="40.64" y="2.54" smashed="yes" rot="R180">
+<attribute name="NAME" x="44.45" y="2.8291" size="1.27" layer="25" rot="R180" align="bottom-center"/>
+</element>
+<element name="R6" library="roomready" library_urn="urn:adsk.eagle:library:9911636" package="R0603" package3d_urn="urn:adsk.eagle:package:7587835/3" value="DNP" x="41.402" y="6.858" smashed="yes" rot="R180">
+<attribute name="NAME" x="41.148" y="10.16" size="1.27" layer="25" rot="R270"/>
 </element>
 </elements>
@@
 <contactref element="R4" pad="2"/>
 <contactref element="OP1" pad="8"/>
-<contactref element="R5" pad="2"/>
 <wire x1="32.6" y1="5.08" x2="30.8113" y2="6.8687" width="0.3048" layer="1"/>
 <wire x1="30.8113" y1="6.8687" x2="30.8113" y2="6.94" width="0.3048" layer="1"/>
-<wire x1="36.78705" y1="5.373" x2="37.719" y2="5.373" width="0.3048" layer="1"/>
-<wire x1="36.52825" y1="5.1142" x2="36.78705" y2="5.373" width="0.3048" layer="1"/>
-<wire x1="32.6" y1="5.08" x2="32.6342" y2="5.1142" width="0.3048" layer="1"/>
-<wire x1="32.6342" y1="5.1142" x2="36.52825" y2="5.1142" width="0.3048" layer="1"/>
+<wire x1="32.6342" y1="5.1142" x2="32.6" y2="5.08" width="0.3048" layer="1"/>
 <contactref element="TP6" pad="P$1"/>
 <wire x1="30.8113" y1="6.94" x2="32.213" y2="6.94" width="0.3048" layer="1"/>
@@
 <wire x1="31.877" y1="11.523" x2="35.56" y2="15.206" width="0.3048" layer="1"/>
 <wire x1="35.56" y1="15.206" x2="35.56" y2="16.51" width="0.3048" layer="1"/>
-</signal>
-<signal name="N$2">
-<contactref element="R5" pad="1"/>
-<contactref element="R6" pad="2"/>
-<wire x1="37.719" y1="7.073" x2="36.957" y2="7.835" width="0.3048" layer="1"/>
-<wire x1="36.957" y1="7.835" x2="36.957" y2="8.548" width="0.3048" layer="1"/>
+<contactref element="R6" pad="1"/>
+<contactref element="J4" pad="P$1"/>
+<wire x1="40.5082" y1="5.1142" x2="32.6342" y2="5.1142" width="0.3048" layer="1"/>
+<wire x1="42.252" y1="6.858" x2="40.5082" y2="5.1142" width="0.3048" layer="1"/>
+<wire x1="40.5082" y1="5.1142" x2="40.5082" y2="3.9418" width="0.3048" layer="1"/>
+<wire x1="40.5082" y1="3.9418" x2="41.91" y2="2.54" width="0.3048" layer="1"/>
 </signal>
 <signal name="LP_FILT">
 <contactref element="C4" pad="1"/>
-<contactref element="R6" pad="1"/>
 <contactref element="OP1" pad="12"/>
-<wire x1="36.957" y1="10.248" x2="36.869" y2="10.16" width="0.3048" layer="1"/>
-<wire x1="36.869" y1="10.16" x2="33.02" y2="10.16" width="0.3048" layer="1"/>
-<wire x1="33.02" y1="10.16" x2="32.385" y2="9.525" width="0.3048" layer="1"/>
+<wire x1="32.385" y1="9.525" x2="33.02" y2="10.16" width="0.3048" layer="1"/>
 <wire x1="32.385" y1="9.525" x2="30.8263" y2="9.525" width="0.3048" layer="1"/>
 <wire x1="30.8263" y1="9.525" x2="30.8113" y2="9.54" width="0.3048" layer="1"/>
-<wire x1="36.957" y1="10.248" x2="39.116" y2="10.248" width="0.3048" layer="1"/>
 <contactref element="TP7" pad="P$1"/>
 <wire x1="40.64" y1="16.51" x2="41.402" y2="15.748" width="0.3048" layer="1"/>
@@
 <wire x1="41.354" y1="9.985" x2="39.379" y2="9.985" width="0.3048" layer="1"/>
 <wire x1="39.379" y1="9.985" x2="39.116" y2="10.248" width="0.3048" layer="1"/>
+<contactref element="R5" pad="2"/>
+<wire x1="36.869" y1="10.16" x2="36.957" y2="10.248" width="0.3048" layer="1"/>
+<wire x1="33.02" y1="10.16" x2="36.869" y2="10.16" width="0.3048" layer="1"/>
+<wire x1="39.116" y1="10.248" x2="36.957" y2="10.248" width="0.3048" layer="1"/>
 </signal>
 <signal name="ENV">
@@
 <wire x1="38.012" y1="11.557" x2="38.52" y2="12.065" width="0.3048" layer="1"/>
 </signal>
+<signal name="N$2">
+<contactref element="J4" pad="P$2"/>
+<contactref element="R5" pad="1"/>
+<contactref element="R6" pad="2"/>
+<wire x1="36.957" y1="7.835" x2="36.957" y2="8.548" width="0.3048" layer="1"/>
+<wire x1="40.552" y1="6.858" x2="39.8279125" y2="6.858" width="0.3048" layer="1"/>
+<wire x1="39.8279125" y1="6.858" x2="39.6529125" y2="6.683" width="0.3048" layer="1"/>
+<wire x1="39.6529125" y1="6.683" x2="39.37" y2="6.683" width="0.3048" layer="1"/>
+<wire x1="39.37" y1="6.683" x2="38.109" y2="6.683" width="0.3048" layer="1"/>
+<wire x1="38.109" y1="6.683" x2="36.957" y2="7.835" width="0.3048" layer="1"/>
+<wire x1="39.37" y1="2.54" x2="39.37" y2="6.35" width="0.3048" layer="16"/>
+<via x="39.37" y="6.35" extent="1-16" drill="0.35"/>
+<wire x1="39.37" y1="6.35" x2="39.37" y2="6.683" width="0.3048" layer="1"/>
+</signal>
 </signals>
