File: Followers/v1/followers_v1.brd (EAGLE design)
At the start: 19 x 108.4 mm, 106 parts, among them IC1 OPA1641, IC14 TL072D, IC2 LM324PW, IC3 LM324PW, IC4 LM324PW, IC5 LM324PW, IC6 LM4040B10, IC7 LM324PW, IC8 LM324PW, IC9 LM324PW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

Commit message: Clean up power section
Parts:
- moved C2 389.2 mm to (1.91, -286.7), turned to 0 degrees
- moved C1 382.6 mm to (1.91, -280.4), turned to 0 degrees
Connections:
- net !GATE: no longer IC9.7
- net ENVELOPE: no longer IC9.6
- net GATE: no longer IC9.1
- net GND: no longer IC9.3
- net N$1: no longer IC9.5
- net N$8: no longer IC9.2
Routing:
- net VEE: track 151.4 -> 0.00 mm, vias 6 -> 0
- net VCC: track 144.3 -> 0.00 mm, vias 7 -> 0
- net AMP_OUT: track 31.8 -> 0.00 mm
- net N$4: track 27.7 -> 0.00 mm
- net N$15: track 22.3 -> 0.00 mm, vias 2 -> 0
- net N$9: track 19.4 -> 0.00 mm
- net N$10: track 4.62 -> 0.00 mm
- net N$6: track 4.47 -> 0.00 mm
- net N$20: track 4.46 -> 0.00 mm
- net N$13: track 4.10 -> 0.00 mm
- net N$3: track 4.07 -> 0.00 mm
- net N$2: track 3.62 -> 0.00 mm
- net N$22: track 1.22 -> 0.00 mm
- net N$44: track 1.18 -> 0.00 mm

Commit message: Fixed op-amps
Parts:
- removed D3: DNP, diode:SOT23
- removed IC14: TL072D, og-linear:SO08
- removed IC5, IC7, IC8: LM324PW, og-ics:TSSOP14
- added C17: 4.7u, rcl:C0603
- added C18: 100n, rcl:C0402
- IC4: value LM324PW -> TL072D; device og-ics:TSSOP14 -> og-linear:SO08
- R7: value 50kB -> 50k
- moved C9 336.1 mm to (0.64, -297.5)
- moved IC4 154.6 mm to (3.81, -160.0)
Connections:
- removed net ENVELOPE: IC7.1, IC7.2
- new net N$27: C17.1, J6.P3
- new net N$32: C17.2, IC2.3
- net AREF_+10: now also IC2.13; no longer IC5.9
- net FULL_WAVE_RECT: now also IC2.12, IC2.8; no longer IC4.14, IC5.10
- net FWR_CLIP: now also IC2.14; no longer IC5.8
- net GND: now also C18.1, C4.1, C6.2, IC4.4; no longer C4.2, C6.1, IC14.4, IC2.11
- net N$100: now also IC4.1; no longer IC14.1
- net N$101: now also IC4.7; no longer IC14.7
- net N$11: now also IC2.6; no longer IC4.9
- net N$12: now also IC2.10; no longer IC4.12
- net N$14: now also IC2.9; no longer IC4.13
- net N$17: now also IC3.13; no longer IC8.6
- net N$19: no longer IC7.3
- net N$2: no longer D3.3
- net N$30: now also IC3.14; no longer IC8.7
- net N$33: now also IC2.1, IC2.2, IC2.5; no longer IC4.10, J6.P3
- net N$5: now also IC2.7; no longer IC4.8
- net N$96: now also IC4.3, IC4.6; no longer IC14.3, IC14.6
- net N$97: now also IC4.2; no longer IC14.2
- net N$99: now also IC4.5; no longer IC14.5
- net SLEW: now also IC3.12; no longer IC8.5
- net V+: no longer IC4.4, IC5.4, IC7.4, IC8.4
- net V-: no longer IC4.11, IC5.11, IC7.11, IC8.11
- net VCC: now also C6.1, IC4.8; no longer C4.1, D3.2, IC14.8
- net VEE: now also C18.2, C4.2, IC2.11; no longer C6.2, D3.1

Commit message: Slew rate limiter
Parts:
- removed JP1, JP3: (no value), SparkFun:1X03
- removed R24: 10k, rcl:R0402
- removed R27: 1.0M, rcl:R0402
- added J11, J4: PJ301_THONKICONN6, og-pj301:WQP_PJ_301M6
- added R18, R19: 50k, og-pots:ALPS_POT_VERTICAL_PS
- C11: value 1u -> 10u
- R23: value 100k -> 510
- R25: value 2.7k -> 100k
- R26: value 20k -> 47k
- R28: value 430k -> 47k
- moved J8 240.0 mm to (3.81, -338.8)
- moved R23 143.8 mm to (0.64, -361.3)
Connections:
- new net LP_DC: J11.P2, R23.1
- new net N$40: J4.P3, R23.2
- new net N$41: J11.P3
- new net N$42: J10.P3
- net FULL_WAVE_RECT: no longer D5.A, D6.C
- net GND: now also IC3.10, IC3.3, IC3.6, J11.P1, J4.P1; no longer C11.2, R27.1
- net N$18: now also IC3.2, R25.2; no longer D5.C, JP1.2
- net N$19: now also IC3.1, R26.1; no longer C11.1, R23.2, R24.2, R25.2, R26.2, R27.2, R28.2
- net N$21: now also IC3.5, R26.2, R28.1; no longer JP3.3, R24.1
- net N$23: now also D5.A, D6.C, IC3.7; no longer JP3.1, R23.1
- net N$24: now also D5.C, R19.P$3; no longer D6.A, JP3.2, R28.1
- net N$25: now also D6.A, R18.P$3; no longer JP1.1, R25.1
- net N$26: now also C11.1, IC3.9, R18.P$2, R19.P$2; no longer JP1.3, R26.1
- net N$29: now also R25.1
- net SLEW: now also C11.2, IC3.8, R28.2

Commit message: bomf
Parts:
- removed JP2: (no value), SparkFun:1X03
- removed R12, R20, R21: 100k, rcl:R0402
- removed R13, R14, R15, R16, R17: 200k, rcl:R0402
- removed R22: 20k, rcl:R0402
- moved C10 109.2 mm to (0.64, -379.4)
Connections:
- removed net !GATE: R15.1, R17.2
- removed net GATE: C10.2, R14.2
- removed net N$1: JP2.2, R16.2, R17.1, R21.1
- removed net N$35: JP2.1, R22.1
- removed net N$36: JP2.3, R20.1
- removed net N$39: R12.1, R13.1
- removed net N$8: C10.1, R13.2, R14.1, R15.2
- net GND: no longer R20.2, R21.2, R22.2
- net VCC: no longer R16.1
- net VEE: no longer R12.2
Changed lines of the file:
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@@
 <attribute name="VALUE" x="3.175" y="-248.3485" size="1.27" layer="27" ratio="10"/>
-</element>
-<element name="R16" library="rcl" package="R0402" value="200k" x="0.635" y="-265.1125" smashed="yes">
-<attribute name="NAME" x="0" y="-264.4775" size="1.27" layer="25"/>
-<attribute name="VALUE" x="0" y="-267.0175" size="1.27" layer="27"/>
-</element>
-<element name="R15" library="rcl" package="R0402" value="200k" x="16.8275" y="-260.0325" smashed="yes">
-<attribute name="NAME" x="16.1925" y="-259.3975" size="1.27" layer="25"/>
-<attribute name="VALUE" x="16.1925" y="-261.9375" size="1.27" layer="27"/>
-</element>
-<element name="R14" library="rcl" package="R0402" value="200k" x="11.43" y="-260.0325" smashed="yes">
-<attribute name="NAME" x="10.795" y="-259.3975" size="1.27" layer="25"/>
-<attribute name="VALUE" x="10.795" y="-261.9375" size="1.27" layer="27"/>
-</element>
-<element name="C10" library="rcl" package="C0402" value="68p" x="0.635" y="-270.1925" smashed="yes">
-<attribute name="NAME" x="0" y="-269.5575" size="1.27" layer="25"/>
-<attribute name="VALUE" x="0" y="-272.0975" size="1.27" layer="27"/>
-</element>
-<element name="R17" library="rcl" package="R0402" value="200k" x="6.0325" y="-265.1125" smashed="yes">
-<attribute name="NAME" x="5.3975" y="-264.4775" size="1.27" layer="25"/>
-<attribute name="VALUE" x="5.3975" y="-267.0175" size="1.27" layer="27"/>
-</element>
-<element name="R21" library="rcl" package="R0402" value="100k" x="16.8275" y="-265.1125" smashed="yes">
-<attribute name="NAME" x="16.1925" y="-264.4775" size="1.27" layer="25"/>
-<attribute name="VALUE" x="16.1925" y="-267.0175" size="1.27" layer="27"/>
-</element>
-<element name="R20" library="rcl" package="R0402" value="100k" x="11.43" y="-265.1125" smashed="yes">
-<attribute name="NAME" x="10.795" y="-264.4775" size="1.27" layer="25"/>
-<attribute name="VALUE" x="10.795" y="-267.0175" size="1.27" layer="27"/>
-</element>
-<element name="R22" library="rcl" package="R0402" value="20k" x="10.16" y="-270.1925" smashed="yes">
-<attribute name="NAME" x="9.525" y="-269.5575" size="1.27" layer="25"/>
-<attribute name="VALUE" x="9.525" y="-272.0975" size="1.27" layer="27"/>
-</element>
-<element name="JP2" library="SparkFun" package="1X03" value="" x="9.8425" y="-252.73" smashed="yes">
-<attribute name="NAME" x="8.4963" y="-250.9012" size="1.27" layer="25" ratio="10"/>
-<attribute name="VALUE" x="8.5725" y="-255.905" size="1.27" layer="27"/>
-</element>
-<element name="R13" library="rcl" package="R0402" value="200k" x="6.0325" y="-260.0325" smashed="yes">
-<attribute name="NAME" x="5.3975" y="-259.3975" size="1.27" layer="25"/>
-<attribute name="VALUE" x="5.3975" y="-261.9375" size="1.27" layer="27"/>
 </element>
 <element name="IC9" library="og-ics" package="TSSOP14" value="LM324PW" x="3.4925" y="-254" smashed="yes">
@@
 <attribute name="VALUE" x="4.7625" y="-272.0975" size="1.27" layer="27"/>
 </element>
-<element name="R12" library="rcl" package="R0402" value="100k" x="0.635" y="-260.0325" smashed="yes">
-<attribute name="NAME" x="0" y="-259.3975" size="1.27" layer="25"/>
-<attribute name="VALUE" x="0" y="-261.9375" size="1.27" layer="27"/>
-</element>
 <element name="C1" library="rcl" package="C1206" value="22u" x="1.905" y="-280.3525" smashed="yes">
 <attribute name="NAME" x="0.635" y="-279.0825" size="1.27" layer="25"/>
@@
 <element name="J11" library="og-pj301" package="WQP_PJ_301M6" value="PJ301_THONKICONN6" x="3.81" y="-369.8875" smashed="yes">
 <attribute name="NAME" x="8.31" y="-374.8875" size="1.27" layer="25" rot="R180"/>
+</element>
+<element name="C10" library="rcl" package="C0402" value="68p" x="0.635" y="-379.4125" smashed="yes">
+<attribute name="NAME" x="0" y="-378.7775" size="1.27" layer="25"/>
+<attribute name="VALUE" x="0" y="-381.3175" size="1.27" layer="27"/>
 </element>
 </elements>
@@
 <contactref element="IC6" pad="2"/>
 <contactref element="R9" pad="2"/>
-<contactref element="R21" pad="2"/>
-<contactref element="R20" pad="2"/>
-<contactref element="R22" pad="2"/>
 <contactref element="R10" pad="1"/>
 <contactref element="C1" pad="2"/>
@@
 <contactref element="J4" pad="P1"/>
 <contactref element="J11" pad="P1"/>
-<wire x1="12.08" y1="-265.1125" x2="17.4775" y2="-265.1125" width="0" layer="19" extent="1-1"/>
-<wire x1="10.81" y1="-270.1925" x2="12.08" y2="-265.1125" width="0" layer="19" extent="1-1"/>
-<wire x1="4.7475" y1="-270.1925" x2="10.81" y2="-270.1925" width="0" layer="19" extent="1-1"/>
+<wire x1="4.7475" y1="-270.1925" x2="1.285" y2="-241.935" width="0" layer="19" extent="1-1"/>
 <wire x1="3.305" y1="-280.3525" x2="4.7475" y2="-270.1925" width="0" layer="19" extent="1-1"/>
 <wire x1="0.505" y1="-286.7025" x2="3.305" y2="-280.3525" width="0" layer="19" extent="1-1"/>
 <wire x1="1.285" y1="-297.4975" x2="0.505" y2="-286.7025" width="0" layer="19" extent="1-1"/>
 <wire x1="-0.015" y1="-302.5775" x2="1.285" y2="-297.4975" width="0" layer="19" extent="1-1"/>
-<wire x1="1.285" y1="-241.935" x2="12.08" y2="-265.1125" width="0" layer="19" extent="1-1"/>
 <wire x1="3.81" y1="-344.4875" x2="-0.015" y2="-302.5775" width="0" layer="19" extent="1-1"/>
 <wire x1="3.81" y1="-357.505" x2="3.81" y2="-344.4875" width="0" layer="19" extent="1-1"/>
@@
 <contactref element="L2" pad="1"/>
 <contactref element="IC3" pad="11"/>
-<contactref element="R12" pad="2"/>
 <contactref element="C2" pad="2"/>
 <contactref element="C4" pad="2"/>
@@
 <wire x1="10.4625" y1="15.5575" x2="13.8303" y2="34.925" width="0" layer="19" extent="1-1"/>
 <wire x1="12.2428" y1="12.065" x2="10.4625" y2="15.5575" width="0" layer="19" extent="1-1"/>
-<wire x1="1.285" y1="-260.0325" x2="12.2428" y2="12.065" width="0" layer="19" extent="1-1"/>
-<wire x1="3.305" y1="-286.7025" x2="1.285" y2="-260.0325" width="0" layer="19" extent="1-1"/>
+<wire x1="3.305" y1="-286.7025" x2="12.2428" y2="12.065" width="0" layer="19" extent="1-1"/>
 <wire x1="1.285" y1="-302.5775" x2="3.305" y2="-286.7025" width="0" layer="19" extent="1-1"/>
 </signal>
@@
 <contactref element="IC4" pad="8"/>
 <contactref element="R3" pad="1"/>
-<contactref element="R16" pad="1"/>
 <contactref element="C1" pad="1"/>
 <contactref element="IC1" pad="7"/>
@@
 <wire x1="13.7975" y1="-159.385" x2="7.5175" y2="-172.085" width="0" layer="19" extent="1-1"/>
 <wire x1="1.905" y1="-157.42" x2="13.7975" y2="-159.385" width="0" layer="19" extent="1-1"/>
-<wire x1="-0.015" y1="-265.1125" x2="5.5" y2="-199.39" width="0" layer="19" extent="1-1"/>
-<wire x1="0.505" y1="-280.3525" x2="-0.015" y2="-265.1125" width="0" layer="19" extent="1-1"/>
+<wire x1="0.505" y1="-280.3525" x2="5.5" y2="-199.39" width="0" layer="19" extent="1-1"/>
 <wire x1="-0.015" y1="-297.4975" x2="0.505" y2="-280.3525" width="0" layer="19" extent="1-1"/>
 <wire x1="6.8072" y1="12.065" x2="1.905" y2="-157.42" width="0" layer="19" extent="1-1"/>
@@
 <wire x1="12.2428" y1="13.335" x2="-0.015" y2="-241.935" width="0" layer="19" extent="1-1"/>
 </signal>
-<signal name="!GATE">
-<contactref element="R15" pad="1"/>
-<contactref element="R17" pad="2"/>
-<wire x1="6.6825" y1="-265.1125" x2="16.1775" y2="-260.0325" width="0" layer="19" extent="1-1"/>
-</signal>
-<signal name="N$35">
-<contactref element="R22" pad="1"/>
-<contactref element="JP2" pad="1"/>
-<wire x1="9.51" y1="-270.1925" x2="9.8425" y2="-252.73" width="0" layer="19" extent="1-1"/>
-</signal>
-<signal name="N$36">
-<contactref element="R20" pad="1"/>
-<contactref element="JP2" pad="3"/>
-<wire x1="10.78" y1="-265.1125" x2="14.9225" y2="-252.73" width="0" layer="19" extent="1-1"/>
-</signal>
-<signal name="N$8">
-<contactref element="C10" pad="1"/>
-<contactref element="R14" pad="1"/>
-<contactref element="R15" pad="2"/>
-<contactref element="R13" pad="2"/>
-<wire x1="6.6825" y1="-260.0325" x2="10.78" y2="-260.0325" width="0" layer="19" extent="1-1"/>
-<wire x1="17.4775" y1="-260.0325" x2="10.78" y2="-260.0325" width="0" layer="19" extent="1-1"/>
-<wire x1="-0.015" y1="-270.1925" x2="6.6825" y2="-260.0325" width="0" layer="19" extent="1-1"/>
-</signal>
 <signal name="N$37">
 <contactref element="LED3" pad="K"/>
@@
 <wire x1="0" y1="-274.955" x2="1.5875" y2="-251.2822" width="0" layer="19" extent="1-1"/>
 </signal>
-<signal name="GATE">
-<contactref element="C10" pad="2"/>
-<contactref element="R14" pad="2"/>
-<wire x1="1.285" y1="-270.1925" x2="12.08" y2="-260.0325" width="0" layer="19" extent="1-1"/>
-</signal>
-<signal name="N$39">
-<contactref element="R12" pad="1"/>
-<contactref element="R13" pad="1"/>
-<wire x1="5.3825" y1="-260.0325" x2="-0.015" y2="-260.0325" width="0" layer="19" extent="1-1"/>
-</signal>
-<signal name="N$1">
-<contactref element="R16" pad="2"/>
-<contactref element="R21" pad="1"/>
-<contactref element="JP2" pad="2"/>
-<contactref element="R17" pad="1"/>
-<wire x1="5.3825" y1="-265.1125" x2="16.1775" y2="-265.1125" width="0" layer="19" extent="1-1"/>
-<wire x1="1.285" y1="-265.1125" x2="5.3825" y2="-265.1125" width="0" layer="19" extent="1-1"/>
-<wire x1="12.3825" y1="-252.73" x2="16.1775" y2="-265.1125" width="0" layer="19" extent="1-1"/>
-</signal>
 <signal name="N$27">
