File: Prototyping Tools/Wizard-Architect's Mana Dock/v1/WAM-D.sch (EAGLE design)
At the start: 0 parts

Commit message: WAM-D progress
Parts:
- added J1, J2: OSTVN02A150, SonicAthame:OSTVN02A150
- added J3, J4: M20-9760246, SonicAthame:M20-9760246
- added J5, J6: HEADER-2X2-F-8.5, SonicAthame:HEADER-2X2-F-8.5
Connections:
- new net N$5: J2.1, J4.1, J4.2, J6.1, J6.2
- new net N$6: J2.2, J4.3, J4.4, J6.3, J6.4
- new net N$7: J1.2, J3.3, J3.4, J5.3, J5.4
- new net N$8: J1.1, J3.1, J3.2, J5.1, J5.2

Commit message: Finalize v1
Parts:
- added J7, J8: M20-9760546, SonicAthame:M20-9760546
Changed lines of the file:
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@@
 <part name="J5" library="SonicAthame" library_urn="urn:adsk.eagle:library:22327399" deviceset="HEADER-2X2-F-8.5" device="" package3d_urn="urn:adsk.eagle:package:10700690/6"/>
 <part name="J6" library="SonicAthame" library_urn="urn:adsk.eagle:library:22327399" deviceset="HEADER-2X2-F-8.5" device="" package3d_urn="urn:adsk.eagle:package:10700690/6"/>
+<part name="J7" library="SonicAthame" library_urn="urn:adsk.eagle:library:22327399" deviceset="M20-9760546" device="" package3d_urn="urn:adsk.eagle:package:22547274/3"/>
+<part name="J8" library="SonicAthame" library_urn="urn:adsk.eagle:library:22327399" deviceset="M20-9760546" device="" package3d_urn="urn:adsk.eagle:package:22547274/3"/>
 </parts>
 <sheets>
@@
 <attribute name="VALUE" x="207.391" y="140.208" size="1.778" layer="95" rot="MR180"/>
 </instance>
+<instance part="J7" gate="G$1" x="246.38" y="144.78" smashed="yes">
+<attribute name="NAME" x="242.951" y="156.972" size="1.778" layer="95"/>
+<attribute name="VALUE" x="242.951" y="129.032" size="1.778" layer="95"/>
+</instance>
+<instance part="J8" gate="G$1" x="264.16" y="144.78" smashed="yes">
+<attribute name="NAME" x="260.731" y="156.972" size="1.778" layer="95"/>
+<attribute name="VALUE" x="260.731" y="129.032" size="1.778" layer="95"/>
+</instance>
 </instances>
