File: Modules/Elementals/Growth/hardware/pcb/growth_v1.sch (EAGLE design)
At the start: 18 parts, among them J1 EURO_POWER, J2 WQP-PJ398SM6, J3 WQP-PJ398SM6, J4 WQP-PJ398SM6, J5 WQP-PJ398SM6, U1 TL072P

Commit message: Finalized(?)
Parts:
- C1, C2: device SonicAthame:CAP_POLLYTIC_H -> SonicAthame:CAP_POLLYTIC_H_R
- R2, R3, R4, R6, R7, R8: device SonicAthame:RESISTOR -> SonicAthame:RESISTOR0207/2V
Changed lines of the file:
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@@
 <schematic xreflabel="%F%N/%S.%C%R" xrefpart="/%S.%C%R">
 <attributes>
+<attribute name="TITLE" value="Elemental Growth"/>
 </attributes>
 <variantdefs>
@@
 <parts>
 <part name="U1" library="SonicAthame" library_urn="urn:adsk.eagle:library:22327399" deviceset="TL072" device="P" package3d_urn="urn:adsk.eagle:package:16409/2"/>
-<part name="FRAME1" library="SonicAthame" library_urn="urn:adsk.eagle:library:22327399" deviceset="FRAME_TABL_L" device=""/>
-<part name="J1" library="SonicAthame" library_urn="urn:adsk.eagle:library:22327399" deviceset="EURO_POWER" device="" package3d_urn="urn:adsk.eagle:package:26183621/2"/>
+<part name="FRAME1" library="SonicAthame" library_urn="urn:adsk.eagle:library:22327399" deviceset="FRAME_TABL_L" device="">
+<attribute name="DOCNUM" value=""/>
+<attribute name="TITLE" value=""/>
+</part>
+<part name="J1" library="SonicAthame" library_urn="urn:adsk.eagle:library:22327399" deviceset="EURO_POWER" device="" package3d_urn="urn:adsk.eagle:package:26183621/3"/>
 <part name="SUPPLY1" library="SonicAthame" library_urn="urn:adsk.eagle:library:22327399" deviceset="+12V" device=""/>
 <part name="SUPPLY2" library="SonicAthame" library_urn="urn:adsk.eagle:library:22327399" deviceset="-12V" device=""/>
@@
 <part name="SUPPLY4" library="SonicAthame" library_urn="urn:adsk.eagle:library:22327399" deviceset="+12V" device=""/>
 <part name="SUPPLY5" library="SonicAthame" library_urn="urn:adsk.eagle:library:22327399" deviceset="-12V" device=""/>
-<part name="R1" library="SonicAthame" library_urn="urn:adsk.eagle:library:22327399" deviceset="ALPHA_POT_VERTICAL" device="VERTICAL" package3d_urn="urn:adsk.eagle:package:22328184/1" value="100k"/>
-<part name="R2" library="SonicAthame" library_urn="urn:adsk.eagle:library:22327399" deviceset="RESISTOR" device="" package3d_urn="urn:adsk.eagle:package:26183828/1" value="1k"/>
-<part name="R3" library="SonicAthame" library_urn="urn:adsk.eagle:library:22327399" deviceset="RESISTOR" device="" package3d_urn="urn:adsk.eagle:package:26183828/1" value="10k"/>
-<part name="R4" library="SonicAthame" library_urn="urn:adsk.eagle:library:22327399" deviceset="RESISTOR" device="" package3d_urn="urn:adsk.eagle:package:26183828/1" value="510"/>
+<part name="R1" library="SonicAthame" library_urn="urn:adsk.eagle:library:22327399" deviceset="ALPHA_POT_VERTICAL" device="VERTICAL" package3d_urn="urn:adsk.eagle:package:22328184/2" value="100k"/>
+<part name="R2" library="SonicAthame" library_urn="urn:adsk.eagle:library:22327399" deviceset="RESISTOR" device="0207/2V" package3d_urn="urn:adsk.eagle:package:26183824/1" value="1k"/>
+<part name="R3" library="SonicAthame" library_urn="urn:adsk.eagle:library:22327399" deviceset="RESISTOR" device="0207/2V" package3d_urn="urn:adsk.eagle:package:26183824/1" value="10k"/>
+<part name="R4" library="SonicAthame" library_urn="urn:adsk.eagle:library:22327399" deviceset="RESISTOR" device="0207/2V" package3d_urn="urn:adsk.eagle:package:26183824/1" value="510"/>
 <part name="SUPPLY6" library="SonicAthame" library_urn="urn:adsk.eagle:library:22327399" deviceset="GND" device=""/>
-<part name="J2" library="SonicAthame" library_urn="urn:adsk.eagle:library:22327399" deviceset="WQP-PJ398SM" device="6" package3d_urn="urn:adsk.eagle:package:22328185/1"/>
+<part name="J2" library="SonicAthame" library_urn="urn:adsk.eagle:library:22327399" deviceset="WQP-PJ398SM" device="6" package3d_urn="urn:adsk.eagle:package:22328185/3"/>
 <part name="SUPPLY7" library="SonicAthame" library_urn="urn:adsk.eagle:library:22327399" deviceset="GND" device=""/>
-<part name="J3" library="SonicAthame" library_urn="urn:adsk.eagle:library:22327399" deviceset="WQP-PJ398SM" device="6" package3d_urn="urn:adsk.eagle:package:22328185/1"/>
+<part name="J3" library="SonicAthame" library_urn="urn:adsk.eagle:library:22327399" deviceset="WQP-PJ398SM" device="6" package3d_urn="urn:adsk.eagle:package:22328185/3"/>
 <part name="SUPPLY8" library="SonicAthame" library_urn="urn:adsk.eagle:library:22327399" deviceset="GND" device=""/>
-<part name="R5" library="SonicAthame" library_urn="urn:adsk.eagle:library:22327399" deviceset="ALPHA_POT_VERTICAL" device="VERTICAL" package3d_urn="urn:adsk.eagle:package:22328184/1" value="10k"/>
-<part name="R6" library="SonicAthame" library_urn="urn:adsk.eagle:library:22327399" deviceset="RESISTOR" device="" package3d_urn="urn:adsk.eagle:package:26183828/1" value="1.1k"/>
-<part name="R7" library="SonicAthame" library_urn="urn:adsk.eagle:library:22327399" deviceset="RESISTOR" device="" package3d_urn="urn:adsk.eagle:package:26183828/1" value="10k"/>
-<part name="R8" library="SonicAthame" library_urn="urn:adsk.eagle:library:22327399" deviceset="RESISTOR" device="" package3d_urn="urn:adsk.eagle:package:26183828/1" value="510"/>
+<part name="R5" library="SonicAthame" library_urn="urn:adsk.eagle:library:22327399" deviceset="ALPHA_POT_VERTICAL" device="VERTICAL" package3d_urn="urn:adsk.eagle:package:22328184/2" value="10k"/>
+<part name="R6" library="SonicAthame" library_urn="urn:adsk.eagle:library:22327399" deviceset="RESISTOR" device="0207/2V" package3d_urn="urn:adsk.eagle:package:26183824/1" value="1.1k"/>
+<part name="R7" library="SonicAthame" library_urn="urn:adsk.eagle:library:22327399" deviceset="RESISTOR" device="0207/2V" package3d_urn="urn:adsk.eagle:package:26183824/1" value="10k"/>
+<part name="R8" library="SonicAthame" library_urn="urn:adsk.eagle:library:22327399" deviceset="RESISTOR" device="0207/2V" package3d_urn="urn:adsk.eagle:package:26183824/1" value="510"/>
 <part name="SUPPLY9" library="SonicAthame" library_urn="urn:adsk.eagle:library:22327399" deviceset="GND" device=""/>
-<part name="J4" library="SonicAthame" library_urn="urn:adsk.eagle:library:22327399" deviceset="WQP-PJ398SM" device="6" package3d_urn="urn:adsk.eagle:package:22328185/1"/>
+<part name="J4" library="SonicAthame" library_urn="urn:adsk.eagle:library:22327399" deviceset="WQP-PJ398SM" device="6" package3d_urn="urn:adsk.eagle:package:22328185/3"/>
 <part name="SUPPLY10" library="SonicAthame" library_urn="urn:adsk.eagle:library:22327399" deviceset="GND" device=""/>
-<part name="J5" library="SonicAthame" library_urn="urn:adsk.eagle:library:22327399" deviceset="WQP-PJ398SM" device="6" package3d_urn="urn:adsk.eagle:package:22328185/1"/>
+<part name="J5" library="SonicAthame" library_urn="urn:adsk.eagle:library:22327399" deviceset="WQP-PJ398SM" device="6" package3d_urn="urn:adsk.eagle:package:22328185/3"/>
 <part name="SUPPLY11" library="SonicAthame" library_urn="urn:adsk.eagle:library:22327399" deviceset="GND" device=""/>
-<part name="C3" library="SonicAthame" library_urn="urn:adsk.eagle:library:22327399" deviceset="CAP_NONPOL" device="025-024X044" package3d_urn="urn:adsk.eagle:package:26183826/1" value="100n"/>
-<part name="C4" library="SonicAthame" library_urn="urn:adsk.eagle:library:22327399" deviceset="CAP_NONPOL" device="025-024X044" package3d_urn="urn:adsk.eagle:package:26183826/1" value="100n"/>
+<part name="C3" library="SonicAthame" library_urn="urn:adsk.eagle:library:22327399" deviceset="CAP_NONPOL" device="025-024X044" package3d_urn="urn:adsk.eagle:package:26183826/2" value="100n"/>
+<part name="C4" library="SonicAthame" library_urn="urn:adsk.eagle:library:22327399" deviceset="CAP_NONPOL" device="025-024X044" package3d_urn="urn:adsk.eagle:package:26183826/2" value="100n"/>
 <part name="SUPPLY12" library="SonicAthame" library_urn="urn:adsk.eagle:library:22327399" deviceset="GND" device=""/>
 <part name="SUPPLY13" library="SonicAthame" library_urn="urn:adsk.eagle:library:22327399" deviceset="GND" device=""/>
-<part name="C1" library="SonicAthame" library_urn="urn:adsk.eagle:library:22327399" deviceset="CAP_POL" device="LYTIC_H" package3d_urn="urn:adsk.eagle:package:26183890/1" value="10u"/>
-<part name="C2" library="SonicAthame" library_urn="urn:adsk.eagle:library:22327399" deviceset="CAP_POL" device="LYTIC_H" package3d_urn="urn:adsk.eagle:package:26183890/1" value="10u"/>
+<part name="C1" library="SonicAthame" library_urn="urn:adsk.eagle:library:22327399" deviceset="CAP_POL" device="LYTIC_H_R" package3d_urn="urn:adsk.eagle:package:26183890/3" value="10u"/>
+<part name="C2" library="SonicAthame" library_urn="urn:adsk.eagle:library:22327399" deviceset="CAP_POL" device="LYTIC_H_R" package3d_urn="urn:adsk.eagle:package:26183890/3" value="10u"/>
 </parts>
 <sheets>
@@
 <attribute name="LAST_DATE_TIME" x="312.42" y="1.27" size="2.54" layer="94"/>
 <attribute name="SHEET" x="386.08" y="1.27" size="2.54" layer="94"/>
+<attribute name="TITLE" x="312.42" y="11.43" size="2.54" layer="94"/>
 </instance>
 <instance part="R1" gate="G$1" x="223.52" y="167.64" smashed="yes" rot="MR270">

Commit message: Better power layout
Parts:
- C1, C2: device SonicAthame:CAP_POLLYTIC_H_R -> SonicAthame:CAP_POLLYTIC_H_L
Changed lines of the file:
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@@
 <part name="SUPPLY12" library="SonicAthame" library_urn="urn:adsk.eagle:library:22327399" deviceset="GND" device=""/>
 <part name="SUPPLY13" library="SonicAthame" library_urn="urn:adsk.eagle:library:22327399" deviceset="GND" device=""/>
-<part name="C1" library="SonicAthame" library_urn="urn:adsk.eagle:library:22327399" deviceset="CAP_POL" device="LYTIC_H_R" package3d_urn="urn:adsk.eagle:package:26183890/3" value="10u"/>
-<part name="C2" library="SonicAthame" library_urn="urn:adsk.eagle:library:22327399" deviceset="CAP_POL" device="LYTIC_H_R" package3d_urn="urn:adsk.eagle:package:26183890/3" value="10u"/>
+<part name="C1" library="SonicAthame" library_urn="urn:adsk.eagle:library:22327399" deviceset="CAP_POL" device="LYTIC_H_L" package3d_urn="urn:adsk.eagle:package:26215121/2" value="10u"/>
+<part name="C2" library="SonicAthame" library_urn="urn:adsk.eagle:library:22327399" deviceset="CAP_POL" device="LYTIC_H_L" package3d_urn="urn:adsk.eagle:package:26215121/2" value="10u"/>
 </parts>
 <sheets>
