File: Modules/Elementals/Growth/hardware/pcb/growth_v2.sch (EAGLE design)
At the start: 20 parts, among them J1 EURO_POWER, J2 WQP-PJ398SM6, J3 WQP-PJ398SM6, J4 WQP-PJ398SM6, J5 WQP-PJ398SM6, U1 TL072P

Commit message: Changed bypass caps to 22p for better HF response. https://northcoastsynthesis.com/news/understanding-stabilization-capacitors/
Parts:
- C5, C6: value 47p -> 22p
Changed lines of the file:
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@@
 <part name="C2" library="SonicAthame" library_urn="urn:adsk.eagle:library:22327399" deviceset="CAP_POL" device="LYTIC_H_L" package3d_urn="urn:adsk.eagle:package:26215121/2" value="10u"/>
 <part name="FRAME1" library="SonicAthame" library_urn="urn:adsk.eagle:library:22327399" deviceset="FRAME_TABL_L" device=""/>
-<part name="C5" library="SonicAthame" library_urn="urn:adsk.eagle:library:22327399" deviceset="CAP_NONPOL" device="050-024X044" package3d_urn="urn:adsk.eagle:package:26183827/3" value="47p"/>
-<part name="C6" library="SonicAthame" library_urn="urn:adsk.eagle:library:22327399" deviceset="CAP_NONPOL" device="050-024X044" package3d_urn="urn:adsk.eagle:package:26183827/3" value="47p"/>
+<part name="C5" library="SonicAthame" library_urn="urn:adsk.eagle:library:22327399" deviceset="CAP_NONPOL" device="050-024X044" package3d_urn="urn:adsk.eagle:package:26183827/3" value="22p"/>
+<part name="C6" library="SonicAthame" library_urn="urn:adsk.eagle:library:22327399" deviceset="CAP_NONPOL" device="050-024X044" package3d_urn="urn:adsk.eagle:package:26183827/3" value="22p"/>
 </parts>
 <sheets>

Commit message: Used more compact components for Elemental Growth
Parts:
- C1, C2: device SonicAthame:CAP_POLLYTIC_H_L -> SonicAthame:CAP_POLLYTIC_V
- C5, C6: device SonicAthame:CAP_NONPOL050-024X044 -> SonicAthame:CAP_NONPOL025-024X044
Changed lines of the file:
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@@
 <parts>
 <part name="U1" library="SonicAthame" library_urn="urn:adsk.eagle:library:22327399" deviceset="TL072" device="P" package3d_urn="urn:adsk.eagle:package:16409/2"/>
-<part name="J1" library="SonicAthame" library_urn="urn:adsk.eagle:library:22327399" deviceset="EURO_POWER" device="" package3d_urn="urn:adsk.eagle:package:26183621/3"/>
+<part name="J1" library="SonicAthame" library_urn="urn:adsk.eagle:library:22327399" deviceset="EURO_POWER" device="" package3d_urn="urn:adsk.eagle:package:26183621/4"/>
 <part name="SUPPLY1" library="SonicAthame" library_urn="urn:adsk.eagle:library:22327399" deviceset="+12V" device=""/>
 <part name="SUPPLY2" library="SonicAthame" library_urn="urn:adsk.eagle:library:22327399" deviceset="-12V" device=""/>
@@
 <part name="SUPPLY12" library="SonicAthame" library_urn="urn:adsk.eagle:library:22327399" deviceset="GND" device=""/>
 <part name="SUPPLY13" library="SonicAthame" library_urn="urn:adsk.eagle:library:22327399" deviceset="GND" device=""/>
-<part name="C1" library="SonicAthame" library_urn="urn:adsk.eagle:library:22327399" deviceset="CAP_POL" device="LYTIC_H_L" package3d_urn="urn:adsk.eagle:package:26215121/2" value="10u"/>
-<part name="C2" library="SonicAthame" library_urn="urn:adsk.eagle:library:22327399" deviceset="CAP_POL" device="LYTIC_H_L" package3d_urn="urn:adsk.eagle:package:26215121/2" value="10u"/>
+<part name="C1" library="SonicAthame" library_urn="urn:adsk.eagle:library:22327399" deviceset="CAP_POL" device="LYTIC_V" package3d_urn="urn:adsk.eagle:package:26183889/3" value="10u"/>
+<part name="C2" library="SonicAthame" library_urn="urn:adsk.eagle:library:22327399" deviceset="CAP_POL" device="LYTIC_V" package3d_urn="urn:adsk.eagle:package:26183889/3" value="10u"/>
 <part name="FRAME1" library="SonicAthame" library_urn="urn:adsk.eagle:library:22327399" deviceset="FRAME_TABL_L" device=""/>
-<part name="C5" library="SonicAthame" library_urn="urn:adsk.eagle:library:22327399" deviceset="CAP_NONPOL" device="050-024X044" package3d_urn="urn:adsk.eagle:package:26183827/3" value="22p"/>
-<part name="C6" library="SonicAthame" library_urn="urn:adsk.eagle:library:22327399" deviceset="CAP_NONPOL" device="050-024X044" package3d_urn="urn:adsk.eagle:package:26183827/3" value="22p"/>
+<part name="C5" library="SonicAthame" library_urn="urn:adsk.eagle:library:22327399" deviceset="CAP_NONPOL" device="025-024X044" package3d_urn="urn:adsk.eagle:package:26183826/2" value="22p"/>
+<part name="C6" library="SonicAthame" library_urn="urn:adsk.eagle:library:22327399" deviceset="CAP_NONPOL" device="025-024X044" package3d_urn="urn:adsk.eagle:package:26183826/2" value="22p"/>
 </parts>
 <sheets>
