File: Modules/Elementals/Center/hardware/pcb/center_v1.brd (EAGLE design)
At the start: 17.8 x 100 mm, 24 parts, among them J1 WQP-PJ398SM6, J10 WQP-PJ398SM6, J11 WQP-PJ398SM6, J12 WQP-PJ398SM6, J2 WQP-PJ398SM6, J3 WQP-PJ398SM6, J4 WQP-PJ398SM6, J5 WQP-PJ398SM6, J6 WQP-PJ398SM6, J7 WQP-PJ398SM6, J8 WQP-PJ398SM6, J9 WQP-PJ398SM6

Commit message: Finished center pcb and panel
Parts:
- moved R4 192.1 mm to (13.3, 45.7)
- moved C4 191.8 mm to (7.62, 45.7)
- moved R5 181.9 mm to (13.3, 30.5)
- moved C5 176.6 mm to (7.62, 30.5)
- moved R3 171.8 mm to (13.3, 61.0)
- moved R6 166.4 mm to (13.3, 15.2)
- moved C6 161.7 mm to (7.62, 15.2)
- moved J10 159.0 mm to (14.0, 22.9)
- moved J7 158.8 mm to (3.81, 38.1)
- moved J8 158.8 mm to (14.0, 38.1)
- moved C3 156.3 mm to (7.62, 61.0)
- moved J6 153.9 mm to (14.0, 53.3)
- moved R2 151.5 mm to (13.3, 76.2)
- moved J9 145.1 mm to (3.81, 22.9)
- moved J11 144.0 mm to (3.81, 7.62)
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Connections:
- removed net N$13: C5.1, J9.P2
- removed net N$14: C5.2, J10.P2, R5.2
- removed net N$15: J10.P1, J9.P1, R5.1
- removed net N$16: C6.1, J11.P2
- removed net N$17: C6.2, J12.P2
- removed net N$18: J11.P1, J12.P1, R6.1, R6.2
- new net GND: J1.P1, J10.P1, J11.P1, J12.P1, J2.P1, J3.P1, J4.P1, J5.P1, J6.P1, J7.P1, J8.P1, J9.P1, R1.2, R2.2, R3.2, R4.2, R5.2, R6.2
- net N$1: now also J1.P3; no longer J1.P2
- net N$10: now also C5.2, J10.P3, R5.1; no longer C4.1, J7.P2
- net N$11: now also C6.2, J12.P3, R6.1; no longer C4.2, J8.P2, R4.2
- net N$12: now also C6.1, J11.P3; no longer J7.P1, J8.P1, R4.1
- net N$2: now also J2.P3, R1.1; no longer J2.P2, R1.2
- net N$3: now also C2.2, J4.P3, R2.1; no longer J1.P1, J2.P1, R1.1
- net N$4: now also J3.P3; no longer J3.P2
- net N$5: now also C3.2, J6.P3, R3.1; no longer C2.2, J4.P2, R2.2
- net N$6: now also C3.1, J5.P3; no longer J3.P1, J4.P1, R2.1
- net N$7: now also C4.1, J7.P3; no longer C3.1, J5.P2
- net N$8: now also C4.2, J8.P3, R4.1; no longer C3.2, J6.P2, R3.2
- net N$9: now also C5.1, J9.P3; no longer J5.P1, J6.P1, R3.1
Routing:
- net N$5: track 0.00 -> 5.39 mm
- net N$3: track 0.00 -> 5.39 mm
- net N$2: track 0.00 -> 5.39 mm
- net N$11: track 0.00 -> 5.39 mm
- net N$10: track 0.00 -> 5.39 mm
- net N$8: track 0.00 -> 5.39 mm
- net N$4: track 0.00 -> 3.23 mm
- net N$1: track 0.00 -> 3.23 mm
- net N$6: track 0.00 -> 3.23 mm
- net N$12: track 0.00 -> 3.23 mm
- net N$9: track 0.00 -> 3.23 mm
- net N$7: track 0.00 -> 3.23 mm
Other:
- board text added: "Elemental Center"
- board text removed: "Elemental Growth"
