File: Modules/Elementals/Center/hardware/pcb/center_v2.sch (EAGLE design)
At the start: 24 parts, among them J1 WQP-PJ398SM6, J10 WQP-PJ398SM6, J11 WQP-PJ398SM6, J12 WQP-PJ398SM6, J2 WQP-PJ398SM6, J3 WQP-PJ398SM6, J4 WQP-PJ398SM6, J5 WQP-PJ398SM6, J6 WQP-PJ398SM6, J7 WQP-PJ398SM6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

Commit message: Updated Elemental Center with more compact parts
Parts:
- C1, C2, C3, C4, C5, C6: device SonicAthame:CAP_NONPOL050-024X044 -> SonicAthame:CAP_NONPOL025-024X044
Changed lines of the file:
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@@
 <part name="R1" library="SonicAthame" library_urn="urn:adsk.eagle:library:22327399" deviceset="RESISTOR" device="0207/2V" package3d_urn="urn:adsk.eagle:package:26183824/1" value="100k"/>
 <part name="J2" library="SonicAthame" library_urn="urn:adsk.eagle:library:22327399" deviceset="WQP-PJ398SM" device="6" package3d_urn="urn:adsk.eagle:package:22328185/3"/>
-<part name="C1" library="SonicAthame" library_urn="urn:adsk.eagle:library:22327399" deviceset="CAP_NONPOL" device="050-024X044" package3d_urn="urn:adsk.eagle:package:26183827/3" value="10u"/>
+<part name="C1" library="SonicAthame" library_urn="urn:adsk.eagle:library:22327399" deviceset="CAP_NONPOL" device="025-024X044" package3d_urn="urn:adsk.eagle:package:26183826/2" value="10u"/>
 <part name="FRAME1" library="SonicAthame" library_urn="urn:adsk.eagle:library:22327399" deviceset="FRAME_TABL_L" device=""/>
 <part name="SUPPLY1" library="SonicAthame" library_urn="urn:adsk.eagle:library:22327399" deviceset="GND" device=""/>
@@
 <part name="R2" library="SonicAthame" library_urn="urn:adsk.eagle:library:22327399" deviceset="RESISTOR" device="0207/2V" package3d_urn="urn:adsk.eagle:package:26183824/1" value="100k"/>
 <part name="J4" library="SonicAthame" library_urn="urn:adsk.eagle:library:22327399" deviceset="WQP-PJ398SM" device="6" package3d_urn="urn:adsk.eagle:package:22328185/3"/>
-<part name="C2" library="SonicAthame" library_urn="urn:adsk.eagle:library:22327399" deviceset="CAP_NONPOL" device="050-024X044" package3d_urn="urn:adsk.eagle:package:26183827/3" value="10u"/>
+<part name="C2" library="SonicAthame" library_urn="urn:adsk.eagle:library:22327399" deviceset="CAP_NONPOL" device="025-024X044" package3d_urn="urn:adsk.eagle:package:26183826/2" value="10u"/>
 <part name="SUPPLY4" library="SonicAthame" library_urn="urn:adsk.eagle:library:22327399" deviceset="GND" device=""/>
 <part name="SUPPLY5" library="SonicAthame" library_urn="urn:adsk.eagle:library:22327399" deviceset="GND" device=""/>
@@
 <part name="R3" library="SonicAthame" library_urn="urn:adsk.eagle:library:22327399" deviceset="RESISTOR" device="0207/2V" package3d_urn="urn:adsk.eagle:package:26183824/1" value="100k"/>
 <part name="J6" library="SonicAthame" library_urn="urn:adsk.eagle:library:22327399" deviceset="WQP-PJ398SM" device="6" package3d_urn="urn:adsk.eagle:package:22328185/3"/>
-<part name="C3" library="SonicAthame" library_urn="urn:adsk.eagle:library:22327399" deviceset="CAP_NONPOL" device="050-024X044" package3d_urn="urn:adsk.eagle:package:26183827/3" value="10u"/>
+<part name="C3" library="SonicAthame" library_urn="urn:adsk.eagle:library:22327399" deviceset="CAP_NONPOL" device="025-024X044" package3d_urn="urn:adsk.eagle:package:26183826/2" value="10u"/>
 <part name="SUPPLY7" library="SonicAthame" library_urn="urn:adsk.eagle:library:22327399" deviceset="GND" device=""/>
 <part name="SUPPLY8" library="SonicAthame" library_urn="urn:adsk.eagle:library:22327399" deviceset="GND" device=""/>
@@
 <part name="R4" library="SonicAthame" library_urn="urn:adsk.eagle:library:22327399" deviceset="RESISTOR" device="0207/2V" package3d_urn="urn:adsk.eagle:package:26183824/1" value="100k"/>
 <part name="J8" library="SonicAthame" library_urn="urn:adsk.eagle:library:22327399" deviceset="WQP-PJ398SM" device="6" package3d_urn="urn:adsk.eagle:package:22328185/3"/>
-<part name="C4" library="SonicAthame" library_urn="urn:adsk.eagle:library:22327399" deviceset="CAP_NONPOL" device="050-024X044" package3d_urn="urn:adsk.eagle:package:26183827/3" value="10u"/>
+<part name="C4" library="SonicAthame" library_urn="urn:adsk.eagle:library:22327399" deviceset="CAP_NONPOL" device="025-024X044" package3d_urn="urn:adsk.eagle:package:26183826/2" value="10u"/>
 <part name="SUPPLY10" library="SonicAthame" library_urn="urn:adsk.eagle:library:22327399" deviceset="GND" device=""/>
 <part name="SUPPLY11" library="SonicAthame" library_urn="urn:adsk.eagle:library:22327399" deviceset="GND" device=""/>
@@
 <part name="R5" library="SonicAthame" library_urn="urn:adsk.eagle:library:22327399" deviceset="RESISTOR" device="0207/2V" package3d_urn="urn:adsk.eagle:package:26183824/1" value="100k"/>
 <part name="J10" library="SonicAthame" library_urn="urn:adsk.eagle:library:22327399" deviceset="WQP-PJ398SM" device="6" package3d_urn="urn:adsk.eagle:package:22328185/3"/>
-<part name="C5" library="SonicAthame" library_urn="urn:adsk.eagle:library:22327399" deviceset="CAP_NONPOL" device="050-024X044" package3d_urn="urn:adsk.eagle:package:26183827/3" value="10u"/>
+<part name="C5" library="SonicAthame" library_urn="urn:adsk.eagle:library:22327399" deviceset="CAP_NONPOL" device="025-024X044" package3d_urn="urn:adsk.eagle:package:26183826/2" value="10u"/>
 <part name="SUPPLY13" library="SonicAthame" library_urn="urn:adsk.eagle:library:22327399" deviceset="GND" device=""/>
 <part name="SUPPLY14" library="SonicAthame" library_urn="urn:adsk.eagle:library:22327399" deviceset="GND" device=""/>
@@
 <part name="R6" library="SonicAthame" library_urn="urn:adsk.eagle:library:22327399" deviceset="RESISTOR" device="0207/2V" package3d_urn="urn:adsk.eagle:package:26183824/1" value="100k"/>
 <part name="J12" library="SonicAthame" library_urn="urn:adsk.eagle:library:22327399" deviceset="WQP-PJ398SM" device="6" package3d_urn="urn:adsk.eagle:package:22328185/3"/>
-<part name="C6" library="SonicAthame" library_urn="urn:adsk.eagle:library:22327399" deviceset="CAP_NONPOL" device="050-024X044" package3d_urn="urn:adsk.eagle:package:26183827/3" value="10u"/>
+<part name="C6" library="SonicAthame" library_urn="urn:adsk.eagle:library:22327399" deviceset="CAP_NONPOL" device="025-024X044" package3d_urn="urn:adsk.eagle:package:26183826/2" value="10u"/>
 <part name="SUPPLY16" library="SonicAthame" library_urn="urn:adsk.eagle:library:22327399" deviceset="GND" device=""/>
 <part name="SUPPLY17" library="SonicAthame" library_urn="urn:adsk.eagle:library:22327399" deviceset="GND" device=""/>
