File: Modules/Elementals/Center/p2/hardware/panel/center_panel.brd (EAGLE design)
At the start: 20 x 128.5 mm, 14 parts

Commit message: center p2 panel done
Routing:
- net N$10: track 0.00 -> 8.76 mm
- net N$27: track 0.00 -> 8.26 mm
- net N$26: track 0.00 -> 8.26 mm
- net N$25: track 0.00 -> 8.26 mm
- net N$24: track 0.00 -> 8.26 mm
- net N$23: track 0.00 -> 8.26 mm
- net N$22: track 0.00 -> 8.26 mm
- net N$7: track 0.00 -> 8.13 mm
- net N$2: track 16.1 -> 8.76 mm
- net N$19: track 0.00 -> 1.26 mm
- net N$18: track 0.00 -> 1.26 mm
- net N$21: track 0.00 -> 1.26 mm
- net N$20: track 0.00 -> 1.26 mm
- net N$1: track 7.31 -> 8.00 mm
Other:
- board text added: "In"
- board text added: "Out"
Changed lines of the file:
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@@
 </layers>
 <board>
-<fusionsync huburn="a.cGVyc29uYWw6dWUyZGY0M2Ex" projecturn="a.cGVyc29uYWw6dWUyZGY0M2ExIzIwMjAwODA5MzIyMjM2MzA2" f3durn="urn:adsk.wipprod:dm.lineage:t9ObxSwbQha4Fn-FaitKzg" pcbguid="d3851583-cf4f-4355-b20e-f6c1576f577a" lastpulledtime="" lastsyncedchangeguid="61ec5c27-2676-56b0-13e2-f8734766109c" latestrevisionid="" lastsyncedrevisionid="" lastboardhashguid="b4c794fe-aee9-9424-cbce-ee8024fe66db" lastpushedtime="2021-01-28T18:07:16Z" linktopcb3d="false"/>
+<fusionsync huburn="a.cGVyc29uYWw6dWUyZGY0M2Ex" projecturn="a.cGVyc29uYWw6dWUyZGY0M2ExIzIwMjAwODA5MzIyMjM2MzA2" f3durn="urn:adsk.wipprod:dm.lineage:ET5NhGXiS0WkGR99PfOD_g" pcbguid="" lastpulledtime="" lastsyncedchangeguid="61ec5c27-2676-56b0-13e2-f8734766109c" latestrevisionid="4c25a131-bf30-4826-a037-8a85f1bd100b" lastsyncedrevisionid="4c25a131-bf30-4826-a037-8a85f1bd100b" lastboardhashguid="7a8cc88c-7343-fad1-cda7-fa2327703569" lastpushedtime="2021-01-29T02:35:36Z" linktopcb3d="true"/>
 <plain>
 <text x="10.16" y="114.935" size="1.778" layer="1" font="vector" align="top-center">Elemental Center</text>
 <text x="10.16" y="114.935" size="1.778" layer="29" font="vector" align="top-center">Elemental Center</text>
 <text x="10.16" y="112.395" size="1.016" layer="25" align="top-center">Prototype 2</text>
-<circle x="5.08" y="13.335" radius="3.81" width="0.1524" layer="1"/>
-<circle x="15.24" y="13.335" radius="3.81" width="0.1524" layer="1"/>
-<circle x="10.16" y="19.05" radius="2.54" width="0.1524" layer="1"/>
+<circle x="5.08" y="13.97" radius="3.81" width="0.1524" layer="1"/>
+<circle x="15.24" y="13.97" radius="3.81" width="0.1524" layer="1"/>
+<circle x="10.16" y="19.685" radius="2.54" width="0.1524" layer="1"/>
+<circle x="10.16" y="8.255" radius="2.54" width="0.1524" layer="1"/>
+<text x="5.08" y="107.95" size="1.778" layer="25" align="bottom-center">In</text>
+<text x="15.24" y="107.95" size="1.778" layer="25" align="bottom-center">Out</text>
+<text x="5.08" y="92.71" size="1.778" layer="25" align="bottom-center">In</text>
+<text x="15.24" y="92.71" size="1.778" layer="25" align="bottom-center">Out</text>
+<text x="5.08" y="77.47" size="1.778" layer="25" align="bottom-center">In</text>
+<text x="15.24" y="77.47" size="1.778" layer="25" align="bottom-center">Out</text>
+<text x="5.08" y="62.23" size="1.778" layer="25" align="bottom-center">In</text>
+<text x="15.24" y="62.23" size="1.778" layer="25" align="bottom-center">Out</text>
+<text x="5.08" y="46.99" size="1.778" layer="25" align="bottom-center">In</text>
+<text x="15.24" y="46.99" size="1.778" layer="25" align="bottom-center">Out</text>
+<text x="5.08" y="31.75" size="1.778" layer="25" align="bottom-center">In</text>
+<text x="15.24" y="31.75" size="1.778" layer="25" align="bottom-center">Out</text>
+<wire x1="5.715" y1="102.235" x2="13.97" y2="102.235" width="1.27" layer="29"/>
+<wire x1="5.715" y1="86.995" x2="13.97" y2="86.995" width="1.27" layer="29"/>
+<wire x1="5.715" y1="71.755" x2="13.97" y2="71.755" width="1.27" layer="29"/>
+<wire x1="5.715" y1="56.515" x2="13.97" y2="56.515" width="1.27" layer="29"/>
+<wire x1="5.715" y1="41.275" x2="13.97" y2="41.275" width="1.27" layer="29"/>
+<wire x1="5.715" y1="26.035" x2="13.97" y2="26.035" width="1.27" layer="29"/>
+<wire x1="5.08" y1="13.97" x2="5.08" y2="25.4" width="0.2032" layer="25"/>
+<wire x1="15.24" y1="13.97" x2="15.24" y2="25.4" width="0.2032" layer="25"/>
+<wire x1="8.509" y1="14.605" x2="8.509" y2="13.97" width="0.2032" layer="25"/>
+<wire x1="8.509" y1="13.97" x2="8.509" y2="13.335" width="0.2032" layer="25"/>
+<wire x1="9.144" y1="14.605" x2="9.144" y2="13.97" width="0.2032" layer="25"/>
+<wire x1="9.144" y1="13.97" x2="9.144" y2="13.335" width="0.2032" layer="25"/>
+<wire x1="12.7" y1="13.97" x2="12.7" y2="12.7" width="0.2032" layer="25"/>
+<wire x1="12.7" y1="12.7" x2="13.081" y2="12.573" width="0.2032" layer="25"/>
+<wire x1="13.081" y1="12.573" x2="12.319" y2="12.319" width="0.2032" layer="25"/>
+<wire x1="12.319" y1="12.319" x2="13.081" y2="12.065" width="0.2032" layer="25"/>
+<wire x1="13.081" y1="12.065" x2="12.319" y2="11.811" width="0.2032" layer="25"/>
+<wire x1="12.319" y1="11.811" x2="12.7" y2="11.684" width="0.2032" layer="25"/>
+<wire x1="12.7" y1="11.684" x2="12.7" y2="11.049" width="0.2032" layer="25"/>
+<wire x1="12.065" y1="11.049" x2="13.335" y2="11.049" width="0.2032" layer="25"/>
+<wire x1="13.081" y1="10.668" x2="12.319" y2="10.668" width="0.2032" layer="25"/>
+<wire x1="12.573" y1="10.287" x2="12.827" y2="10.287" width="0.2032" layer="25"/>
+<wire x1="5.08" y1="13.97" x2="8.509" y2="13.97" width="0.2032" layer="25"/>
+<wire x1="9.144" y1="13.97" x2="12.7" y2="13.97" width="0.2032" layer="25"/>
+<wire x1="12.7" y1="13.97" x2="15.24" y2="13.97" width="0.2032" layer="25"/>
+<circle x="12.7" y="13.97" radius="0.254" width="0.508" layer="25"/>
 </plain>
 <attributes>
@@
 <signals>
 <signal name="N$3">
-<wire x1="3.81" y1="15.875" x2="2.54" y2="15.875" width="0.1524" layer="1" curve="-180"/>
+<wire x1="3.81" y1="16.51" x2="2.54" y2="16.51" width="0.1524" layer="1" curve="-180"/>
 </signal>
 <signal name="N$4">
-<wire x1="3.81" y1="15.875" x2="5.08" y2="15.875" width="0.1524" layer="1" curve="-180"/>
+<wire x1="3.81" y1="16.51" x2="5.08" y2="16.51" width="0.1524" layer="1" curve="-180"/>
 </signal>
 <signal name="N$5">
-<wire x1="6.35" y1="15.875" x2="5.08" y2="15.875" width="0.1524" layer="1" curve="-180"/>
+<wire x1="6.35" y1="16.51" x2="5.08" y2="16.51" width="0.1524" layer="1" curve="-180"/>
 </signal>
 <signal name="N$6">
-<wire x1="2.4638" y1="16.0782" x2="2.54" y2="15.875" width="0.1524" layer="1" curve="-36.869898"/>
+<wire x1="2.4638" y1="16.7132" x2="2.54" y2="16.51" width="0.1524" layer="1" curve="-36.869898"/>
 </signal>
 <signal name="N$8">
-<wire x1="7.62" y1="15.875" x2="8.382" y2="15.24" width="0.1524" layer="1" curve="100"/>
+<wire x1="7.62" y1="16.51" x2="8.382" y2="15.875" width="0.1524" layer="1" curve="100"/>
 </signal>
 <signal name="N$9">
-<wire x1="2.54" y1="15.875" x2="2.4638" y2="16.0782" width="0.1524" layer="1" curve="30"/>
+<wire x1="2.54" y1="16.51" x2="2.4638" y2="16.7132" width="0.1524" layer="1" curve="30"/>
 </signal>
 <signal name="N$11">
-<wire x1="6.35" y1="15.875" x2="7.62" y2="15.875" width="0.1524" layer="1" curve="-180"/>
+<wire x1="6.35" y1="16.51" x2="7.62" y2="16.51" width="0.1524" layer="1" curve="-180"/>
 </signal>
 <signal name="N$12">
-<wire x1="13.97" y1="13.335" x2="15.24" y2="13.335" width="0.1524" layer="1" curve="-180"/>
+<wire x1="13.97" y1="13.97" x2="15.24" y2="13.97" width="0.1524" layer="1" curve="-180"/>
 </signal>
 <signal name="N$13">
-<wire x1="16.51" y1="13.335" x2="15.24" y2="13.335" width="0.1524" layer="1" curve="-180"/>
+<wire x1="16.51" y1="13.97" x2="15.24" y2="13.97" width="0.1524" layer="1" curve="-180"/>
 </signal>
 <signal name="N$14">
-<wire x1="13.97" y1="13.335" x2="12.7" y2="13.335" width="0.1524" layer="1" curve="-180"/>
+<wire x1="13.97" y1="13.97" x2="12.7" y2="13.97" width="0.1524" layer="1" curve="-180"/>
 </signal>
 <signal name="N$15">
-<wire x1="16.51" y1="13.335" x2="17.78" y2="13.335" width="0.1524" layer="1" curve="-180"/>
+<wire x1="16.51" y1="13.97" x2="17.78" y2="13.97" width="0.1524" layer="1" curve="-180"/>
 </signal>
 <signal name="N$16">
-<wire x1="11.43" y1="13.335" x2="12.7" y2="13.335" width="0.1524" layer="1" curve="-180"/>
+<wire x1="11.43" y1="13.97" x2="12.7" y2="13.97" width="0.1524" layer="1" curve="-180"/>
 </signal>
 <signal name="N$17">
-<wire x1="19.05" y1="13.335" x2="17.78" y2="13.335" width="0.1524" layer="1" curve="-180"/>
+<wire x1="19.05" y1="13.97" x2="17.78" y2="13.97" width="0.1524" layer="1" curve="-180"/>
+</signal>
+<signal name="N$2">
+<wire x1="10.16" y1="17.145" x2="12.319" y2="20.955" width="0.1524" layer="1"/>
+<wire x1="10.16" y1="17.145" x2="8.001" y2="20.955" width="0.1524" layer="1"/>
 </signal>
 <signal name="N$1">
-<wire x1="7.62" y1="19.05" x2="5.08" y2="25.908" width="0.1524" layer="1"/>
-</signal>
-<signal name="N$2">
-<wire x1="12.7" y1="19.05" x2="15.24" y2="25.908" width="0.1524" layer="1"/>
-<wire x1="12.7" y1="19.05" x2="8.89" y2="21.209" width="0.1524" layer="1"/>
-<wire x1="12.7" y1="19.05" x2="8.89" y2="16.891" width="0.1524" layer="1"/>
+<wire x1="5.08" y1="17.78" x2="5.08" y2="25.781" width="0.1524" layer="1"/>
+</signal>
+<signal name="N$7">
+<wire x1="15.24" y1="17.78" x2="15.24" y2="25.908" width="0.1524" layer="1"/>
+</signal>
+<signal name="N$10">
+<wire x1="10.16" y1="10.795" x2="8.001" y2="6.985" width="0.1524" layer="1"/>
+<wire x1="10.16" y1="10.795" x2="12.319" y2="6.985" width="0.1524" layer="1"/>
+</signal>
+<signal name="N$19">
+<wire x1="8.4582" y1="10.1854" x2="7.5692" y2="11.0744" width="0.1524" layer="1"/>
+</signal>
+<signal name="N$18">
+<wire x1="11.8618" y1="10.1854" x2="12.7508" y2="11.0744" width="0.1524" layer="1"/>
+</signal>
+<signal name="N$20">
+<wire x1="11.8618" y1="17.7546" x2="12.7508" y2="16.8656" width="0.1524" layer="1"/>
+</signal>
+<signal name="N$21">
+<wire x1="8.4582" y1="17.7546" x2="7.5692" y2="16.8656" width="0.1524" layer="1"/>
+</signal>
+<signal name="N$22">
+<wire x1="5.715" y1="102.235" x2="13.97" y2="102.235" width="1.27" layer="1"/>
+</signal>
+<signal name="N$23">
+<wire x1="5.715" y1="86.995" x2="13.97" y2="86.995" width="1.27" layer="1"/>
+</signal>
+<signal name="N$24">
+<wire x1="5.715" y1="71.755" x2="13.97" y2="71.755" width="1.27" layer="1"/>
+</signal>
+<signal name="N$25">
+<wire x1="5.715" y1="56.515" x2="13.97" y2="56.515" width="1.27" layer="1"/>
+</signal>
+<signal name="N$26">
+<wire x1="5.715" y1="41.275" x2="13.97" y2="41.275" width="1.27" layer="1"/>
+</signal>
+<signal name="N$27">
+<wire x1="5.715" y1="26.035" x2="13.97" y2="26.035" width="1.27" layer="1"/>
 </signal>
 </signals>
